File: trx/pcb/pcb.kicad_sch (KiCad schematic)
At the start: 40 parts, among them J1 USB_C, U1 RP2040, U2 W25Q128JVS, U3 TPS56339DDC, Y1 12MHz

Commit message: Update design
Parts:
- removed JP1: VUSB_VCC, Jumper:SolderJumper-2_P1.3mm_Bridged2Bar_RoundedPad1.0x1.5mm, symbol Jumper:SolderJumper_2_Bridged
- removed JP2: VEXT_VCC, Jumper:SolderJumper-2_P1.3mm_Open_RoundedPad1.0x1.5mm, symbol Jumper:SolderJumper_2_Open
- added D1: UHF_ACT, LED_SMD:LED_0805_2012Metric_Pad1.15x1.40mm_HandSolder, symbol Device:LED
- added D2: SBAND_ACT, LED_SMD:LED_0805_2012Metric_Pad1.15x1.40mm_HandSolder, symbol Device:LED
- added J3: SWDIO, Connector_PinHeader_2.54mm:PinHeader_1x04_P2.54mm_Vertical, symbol Connector_Generic:Conn_01x04
- added J4: Ext Power, Connector_PinSocket_2.54mm:PinSocket_1x02_P2.54mm_Vertical, symbol Connector_Generic:Conn_01x02
- added J5: I2C, Connector_PinHeader_2.54mm:PinHeader_1x04_P2.54mm_Vertical, symbol Connector_Generic:Conn_01x04
- added R10, R9: 0, Resistor_SMD:R_0805_2012Metric_Pad1.20x1.40mm_HandSolder, symbol Device:R
- added R11, R13: 10k, Resistor_SMD:R_0603_1608Metric_Pad0.98x0.95mm_HandSolder, symbol Device:R
- added R12, R16, R17: 1k, Resistor_SMD:R_0603_1608Metric_Pad0.98x0.95mm_HandSolder, symbol Device:R
- added R14, R15: 5.1k, Resistor_SMD:R_0603_1608Metric_Pad0.98x0.95mm_HandSolder, symbol Device:R
- added SW1: RESET, Button_Switch_SMD:SW_Push_1P1T_NO_CK_KSC6xxJ, symbol Switch:SW_Push
- added SW2: BOOT, Button_Switch_SMD:SW_Push_1P1T_NO_CK_KSC6xxJ, symbol Switch:SW_Push
Connections:
- net +3V3: now also J3.2 (Pin_2), J5.1 (Pin_1), R11.2, R13.2, R14.2, R15.1
- net FLASH_CS: now also R12.2, R13.1
- net GND: now also D1.1 (K), D2.1 (K), J3.1 (Pin_1), J4.1 (Pin_1), J5.2 (Pin_2), SW1.1, SW2.1
- net SWCLK: now also J3.3 (Pin_3)
- net SWDIO: now also J3.4 (Pin_4)
- net VBUS: now also R9.1
- net VCC: now also R10.2, R9.2
- net VEXT: now also J4.2 (Pin_2), R10.1
- net SPI1_MISO: now reaches U1.11 (GPIO8)
- net SPI1_CS: now reaches U1.12 (GPIO9)
- net SPI1_SCLK: now reaches U1.13 (GPIO10)
- net SPI1_MOSI: now reaches U1.14 (GPIO11)
- net SB_DIO2: now reaches U1.15 (GPIO12)
- net SB_DIO3: now reaches U1.16 (GPIO13)
- net SB_DIO1: now reaches U1.17 (GPIO14)
- net SB_BUSY: now reaches U1.18 (GPIO15)
- net SDA: now reaches U1.2 (GPIO0)
- net SDA: now also J5.4 (Pin_4), R14.1
- net RUN: now reaches U1.26 (RUN)
- net RUN: now also R11.1, SW1.2
- net SPI0_MISO: now reaches U1.27 (GPIO16)
- net SPI0_CS: now reaches U1.28 (GPIO17)
- net SPI0_SCLK: now reaches U1.29 (GPIO18)
- net SCL: now reaches U1.3 (GPIO1)
- net SCL: now also J5.3 (Pin_3), R15.2
- net SPI0_MOSI: now reaches U1.30 (GPIO19)
- net U_RST: now reaches U1.31 (GPIO20)
- net U_BUSY: now reaches U1.32 (GPIO21)
- net LED_UHF: now reaches U1.36 (GPIO24)
- net LED_UHF: now also R16.2
- net LED_SBAND: now reaches U1.37 (GPIO25)
- net LED_SBAND: now also R17.2
- net SB_TXEN: now reaches U1.4 (GPIO2)
- net U_DIO1: now reaches U1.5 (GPIO3)
- net U_DIO2: now reaches U1.6 (GPIO4)
- net U_TXEN: now reaches U1.7 (GPIO5)
- net U_RXEN: now reaches U1.8 (GPIO6)
- net SB_RST: now reaches U1.9 (GPIO7)
- new net: R12.1, SW2.2
- new net: D1.2 (A), R16.1
- new net: D2.2 (A), R17.1
Other:
- sheet radio ports: added SB_BUSY, SB_DIO1, SB_DIO2, SB_DIO3, SB_RST, SB_TXEN, U_BUSY, U_CS, U_DIO1, U_DIO2, U_MISO, U_MOSI, U_RST, U_RXEN, U_SCLK, U_TXEN; removed none
- note added: "Misc"
- note added: "Mounting holes"
- note added: "RF part"
- note added: "SWDIO"
- moved on the sheet: C1, C10, C11, C12, C13, C14, C15, C16, C17, C18, C19, C2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
