File: trx/pcb/radio.kicad_sch (KiCad schematic)
At the start: 9 parts, among them J2 SB_U.FL, U4 SX1280IMLTRT, U5 RFX2401C, Y2 52MHz TCXO

Commit message: Update
Parts:
- added U6: E22-900M22S, E22-900M22S:E22-900M22S, symbol E22-900M22S:E22-900M22S
Connections:
- net +3V3: now also U6.9 (VCC)
- net GND: now also U6.1 (GND), U6.10 (GND), U6.11 (GND), U6.12 (GND), U6.2 (GND), U6.20 (GND), U6.22 (GND), U6.3 (GND), U6.4 (GND), U6.5 (GND)

Commit message: Update design
Parts:
- added C24: 22u, Capacitor_SMD:C_0603_1608Metric_Pad1.08x0.95mm_HandSolder, symbol Device:C
- added C25, C26, C27, C28, C29, C30, C32: 100n, Capacitor_SMD:C_0603_1608Metric_Pad1.08x0.95mm_HandSolder, symbol Device:C
- added C31: 1u, Capacitor_SMD:C_0603_1608Metric_Pad1.08x0.95mm_HandSolder, symbol Device:C
- added L3: 15u, Inductor_SMD:L_0805_2012Metric_Pad1.15x1.40mm_HandSolder, symbol Device:L
- U6: value E22-900M22S -> E22-400M22S
Connections:
- net SB_RXEN is gone; now on net +3V3: U5.6 (RXEN)
- net +3V3: now also U4.11 (VBAT_IO), U4.15 (VBAT), C24.1, C25.2, C26.1, C27.1, C30.1, C32.1
- net GND: now also C24.2, C25.1, C26.2, C27.2, C28.1, C29.1, C30.2, C31.2, C32.2
- net at U4.1 (VR_PA): now also C28.2
- net DCC: now reaches U4.12 (DCC_FB)
- net DCC: now also U4.2 (VDD_IN), C29.2, C31.1, L3.2
- net at U4.14 (DCC_SW): now also L3.1
- net SB_RST: now reaches U4.3 (NRESET)
- net U_DIO1: now reaches U6.13 (DIO1)
- net U_BUSY: now reaches U6.14 (BUSY)
- net U_RST: now reaches U6.15 (NRST)
- net U_MISO: now reaches U6.16 (MISO)
- net U_MOSI: now reaches U6.17 (MOSI)
- net U_SCLK: now reaches U6.18 (SCK)
- net U_CS: now reaches U6.19 (NSS)
- net U_RXEN: now reaches U6.6 (RXEN)
- net U_TXEN: now reaches U6.7 (TXEN)
- net U_DIO2: now reaches U6.8 (DIO2)
- no-connect marks 2 -> 3
Other:
- moved on the sheet: C21, Y2
