File: trx/pcb/pcb.kicad_pcb (KiCad board)
At the start: 4 copper layers, 50 x 50 mm, 50 parts, among them J1 USB_C, J2 SB_U.FL, U1 RP2040, U2 W25Q128JVS, U3 TPS56339DDC, U4 SX1280IMLTRT, U5 RFX2401C, U6 E22-400M30S, Y1 12MHz, Y2 52MHz TCXO

Commit message: Update
Parts:
- U6: value E22-400M30S -> E22-900M22S; footprint E22-900M30S:XCVR_E22-900M30S -> E22-900M22S:E22-900M22S
- moved U6 43.1 mm to (143.1, 72.9)
- renumbered U4 to U1
Connections:
- U1 pad 10: unconnected-(U4-DIO3-Pad10) -> /radio/SB_DIO3
- U1 pad 7: unconnected-(U4-BUSY-Pad7) -> /radio/SB_BUSY
- U1 pad 8: unconnected-(U4-DIO1-Pad8) -> /radio/SB_DIO1
- U1 pad 9: unconnected-(U4-DIO2-Pad9) -> /radio/SB_DIO2
- U6 pad 1: Net-(U6-GND-Pad1) -> GND
- U6 pad 10: Net-(U6-VCC-Pad10) -> GND
- U6 pad 11: Net-(U6-GND-Pad1) -> GND
- U6 pad 12: Net-(U6-GND-Pad1) -> GND
- U6 pad 2: Net-(U6-GND-Pad1) -> GND
- U6 pad 20: Net-(U6-GND-Pad1) -> GND
- U6 pad 22: Net-(U6-GND-Pad1) -> GND
- U6 pad 3: Net-(U6-GND-Pad1) -> GND
- U6 pad 4: Net-(U6-GND-Pad1) -> GND
- U6 pad 5: Net-(U6-GND-Pad1) -> GND
- U6 pad 9: Net-(U6-VCC-Pad10) -> +3V3
Routing:
- net Net-(U3-SW): track 8.28 -> 3.58 mm
- added copper zone on F.Cu, net Net-(U3-SW)

Commit message: Update design
Parts:
- removed JP1: VUSB_VCC, Jumper:SolderJumper-2_P1.3mm_Bridged2Bar_RoundedPad1.0x1.5mm
- removed JP2: VEXT_VCC, Jumper:SolderJumper-2_P1.3mm_Open_RoundedPad1.0x1.5mm
- added C24: 22u, Capacitor_SMD:C_0603_1608Metric_Pad1.08x0.95mm_HandSolder, F.Cu at (134.2, 80.8)
- added C25: 100n, Capacitor_SMD:C_0603_1608Metric_Pad1.08x0.95mm_HandSolder, F.Cu at (134.2, 79.1)
- added C26: 100n, Capacitor_SMD:C_0603_1608Metric_Pad1.08x0.95mm_HandSolder, F.Cu at (143.9, 69.9)
- added C27: 100n, Capacitor_SMD:C_0603_1608Metric_Pad1.08x0.95mm_HandSolder, F.Cu at (143.9, 71.5)
- added C28: 100n, Capacitor_SMD:C_0603_1608Metric_Pad1.08x0.95mm_HandSolder, F.Cu at (143.5, 75.2)
- added C29: 100n, Capacitor_SMD:C_0603_1608Metric_Pad1.08x0.95mm_HandSolder, F.Cu at (143.5, 76.8)
- added C30: 100n, Capacitor_SMD:C_0603_1608Metric_Pad1.08x0.95mm_HandSolder, F.Cu at (153.3, 77.6)
- added C31: 1u, Capacitor_SMD:C_0603_1608Metric_Pad1.08x0.95mm_HandSolder, F.Cu at (150.2, 83.2)
- added C32: 100n, Capacitor_SMD:C_0603_1608Metric_Pad1.08x0.95mm_HandSolder, F.Cu at (148.6, 83.2)
- added D1: UHF_ACT, LED_SMD:LED_0805_2012Metric_Pad1.15x1.40mm_HandSolder, F.Cu at (144.1, 89.9)
- added D2: SBAND_ACT, LED_SMD:LED_0805_2012Metric_Pad1.15x1.40mm_HandSolder, F.Cu at (146.5, 89.9)
- added J3: SWDIO, Connector_PinHeader_2.54mm:PinHeader_1x04_P2.54mm_Vertical, F.Cu at (112.3, 77.1)
- added J4: Ext Power, Connector_PinSocket_2.54mm:PinSocket_1x02_P2.54mm_Vertical, F.Cu at (131.4, 106.8)
- added J5: I2C, Connector_PinHeader_2.54mm:PinHeader_1x04_P2.54mm_Vertical, F.Cu at (143.7, 97.6)
- added L3: 15u, Inductor_SMD:L_0805_2012Metric_Pad1.15x1.40mm_HandSolder, F.Cu at (152.4, 80.3)
- added R10: 0, Resistor_SMD:R_0805_2012Metric_Pad1.20x1.40mm_HandSolder, F.Cu at (133.9, 103.2)
- added R11: 10k, Resistor_SMD:R_0603_1608Metric_Pad0.98x0.95mm_HandSolder, F.Cu at (152.0, 85.1)
- added R12: 1k, Resistor_SMD:R_0603_1608Metric_Pad0.98x0.95mm_HandSolder, F.Cu at (150.9, 93.0)
- added R13: 10k, Resistor_SMD:R_0603_1608Metric_Pad0.98x0.95mm_HandSolder, F.Cu at (132.5, 90.9)
- added R14: 5.1k, Resistor_SMD:R_0603_1608Metric_Pad0.98x0.95mm_HandSolder, F.Cu at (139.7, 93.3)
- added R15: 5.1k, Resistor_SMD:R_0603_1608Metric_Pad0.98x0.95mm_HandSolder, F.Cu at (139.7, 94.8)
- added R16: 1k, Resistor_SMD:R_0603_1608Metric_Pad0.98x0.95mm_HandSolder, F.Cu at (141.2, 88.4)
- added R17: 1k, Resistor_SMD:R_0603_1608Metric_Pad0.98x0.95mm_HandSolder, F.Cu at (149.1, 89.7)
- added R9: 0, Resistor_SMD:R_0805_2012Metric_Pad1.20x1.40mm_HandSolder, F.Cu at (130.9, 103.2)
- added SW1: RESET, Button_Switch_SMD:SW_Push_1P1T_NO_CK_KSC6xxJ, F.Cu at (156.2, 86.8)
- added SW2: BOOT, Button_Switch_SMD:SW_Push_1P1T_NO_CK_KSC6xxJ, F.Cu at (156.2, 96.8)
- U6: value E22-900M22S -> E22-400M22S
- moved U4 31.5 mm to (148.3, 78.2)
- moved L2 31.4 mm to (148.7, 73.4)
- moved C22 31.4 mm to (147.5, 74.4)
- moved C21 31.2 mm to (143.5, 78.5)
- moved Y2 31.2 mm to (143.3, 80.9)
- moved U5 27.4 mm to (148.5, 70.2), turned to 90 degrees
- moved C23 24.5 mm to (149.6, 66.8), turned to 0 degrees
- moved FL1 21.7 mm to (147.1, 64.1), turned to 180 degrees
- moved J2 20.9 mm to (141.8, 64.1)
- moved U6 15.6 mm to (127.9, 69.2), turned to -90 degrees
- moved R1 0.54 mm to (120.5, 82.3)
- moved C3 0.45 mm to (132.5, 92.5)
- moved C12 0.45 mm to (117.3, 82.4)
- moved C19 0.45 mm to (119.0, 82.4)
- moved Y1 0.45 mm to (124.0, 80.8)
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- renumbered U1 to U4
Connections:
- U1 pad 11: unconnected-(U1-GPIO8-Pad11) -> SPI1_MISO
- U1 pad 12: unconnected-(U1-GPIO9-Pad12) -> SPI1_CS
- U1 pad 13: unconnected-(U1-GPIO10-Pad13) -> SPI1_SCLK
- U1 pad 14: unconnected-(U1-GPIO11-Pad14) -> SPI1_MOSI
- U1 pad 15: unconnected-(U1-GPIO12-Pad15) -> SB_DIO2
- U1 pad 16: unconnected-(U1-GPIO13-Pad16) -> SB_DIO3
- U1 pad 17: unconnected-(U1-GPIO14-Pad17) -> SB_DIO1
- U1 pad 18: unconnected-(U1-GPIO15-Pad18) -> SB_BUSY
- U1 pad 2: unconnected-(U1-GPIO0-Pad2) -> SDA
- U1 pad 26: unconnected-(U1-RUN-Pad26) -> RUN
- U1 pad 27: unconnected-(U1-GPIO16-Pad27) -> SPI0_MISO
- U1 pad 28: unconnected-(U1-GPIO17-Pad28) -> SPI0_CS
- U1 pad 29: unconnected-(U1-GPIO18-Pad29) -> SPI0_SCLK
- U1 pad 3: unconnected-(U1-GPIO1-Pad3) -> SCL
- U1 pad 30: unconnected-(U1-GPIO19-Pad30) -> SPI0_MOSI
- U1 pad 31: unconnected-(U1-GPIO20-Pad31) -> U_RST
- U1 pad 32: unconnected-(U1-GPIO21-Pad32) -> U_BUSY
- U1 pad 36: unconnected-(U1-GPIO24-Pad36) -> LED_UHF
- U1 pad 37: unconnected-(U1-GPIO25-Pad37) -> LED_SBAND
- U1 pad 4: unconnected-(U1-GPIO2-Pad4) -> SB_TXEN
- U1 pad 5: unconnected-(U1-GPIO3-Pad5) -> U_DIO1
- U1 pad 6: unconnected-(U1-GPIO4-Pad6) -> U_DIO2
- U1 pad 7: unconnected-(U1-GPIO5-Pad7) -> U_TXEN
- U1 pad 8: unconnected-(U1-GPIO6-Pad8) -> U_RXEN
- U1 pad 9: unconnected-(U1-GPIO7-Pad9) -> SB_RST
- U4 pad 1: unconnected-(U4-VR_PA-Pad1) -> Net-(U4-VR_PA)
- U4 pad 10: /radio/SB_DIO3 -> SB_DIO3
- U4 pad 11: unconnected-(U4-VBAT_IO-Pad11) -> +3V3
- U4 pad 12: unconnected-(U4-DCC_FB-Pad12) -> DCC
- U4 pad 14: unconnected-(U4-DCC_SW-Pad14) -> Net-(U4-DCC_SW)
- U4 pad 15: unconnected-(U4-VBAT-Pad15) -> +3V3
- U4 pad 16: /radio/SB_MISO -> SPI1_MISO
- U4 pad 17: /radio/SB_MOSI -> SPI1_MOSI
- U4 pad 18: /radio/SB_SCLK -> SPI1_SCLK
- U4 pad 19: /radio/SB_CS -> SPI1_CS
- U4 pad 2: unconnected-(U4-VDD_IN-Pad2) -> DCC
- U4 pad 3: unconnected-(U4-NRESET-Pad3) -> SB_RST
- U4 pad 7: /radio/SB_BUSY -> SB_BUSY
- U4 pad 8: /radio/SB_DIO1 -> SB_DIO1
- U4 pad 9: /radio/SB_DIO2 -> SB_DIO2
- U5 pad 5: /radio/SB_TXEN -> SB_TXEN
- U5 pad 6: /radio/SB_RXEN -> +3V3
- U6 pad 13: unconnected-(U6-DIO1-Pad13) -> U_DIO1
- U6 pad 14: unconnected-(U6-BUSY-Pad14) -> U_BUSY
- U6 pad 15: unconnected-(U6-NRST-Pad15) -> U_RST
- U6 pad 16: unconnected-(U6-MISO-Pad16) -> SPI0_MISO
- U6 pad 17: unconnected-(U6-MOSI-Pad17) -> SPI0_MOSI
- U6 pad 18: unconnected-(U6-SCK-Pad18) -> SPI0_SCLK
- U6 pad 19: unconnected-(U6-NSS-Pad19) -> SPI0_CS
- U6 pad 6: unconnected-(U6-RXEN-Pad6) -> U_RXEN
- U6 pad 7: unconnected-(U6-TXEN-Pad7) -> U_TXEN
- U6 pad 8: unconnected-(U6-DIO2-Pad8) -> U_DIO2
Routing:
- net SB_TXEN: track 0.00 -> 58.3 mm
- net RUN: track 0.00 -> 46.9 mm, vias 0 -> 2
- net SPI1_SCLK: track 0.00 -> 44.5 mm, vias 0 -> 2
- net SPI1_CS: track 0.00 -> 44.4 mm, vias 0 -> 4
- net SPI1_MISO: track 0.00 -> 42.8 mm, vias 0 -> 2
- net U_DIO1: track 0.00 -> 41.1 mm, vias 0 -> 2
- net SPI1_MOSI: track 0.00 -> 39.0 mm, vias 0 -> 2
- net LED_SBAND: track 0.00 -> 37.3 mm, vias 0 -> 2
- net SPI0_MOSI: track 0.00 -> 36.2 mm
- net U_BUSY: track 0.00 -> 35.0 mm, vias 0 -> 2
- net U_RST: track 0.00 -> 33.9 mm, vias 0 -> 2
- net SB_RST: track 0.00 -> 33.4 mm, vias 0 -> 2
- net SPI0_SCLK: track 0.00 -> 33.2 mm
- net SPI0_MISO: track 0.00 -> 33.2 mm
- net SB_DIO3: track 0.00 -> 31.2 mm, vias 0 -> 2
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- added copper zone on F.Cu, net DCC
Other:
- board text added: "12V"
- board text added: "3V3"
- board text added: "3V3 GND SCL SDA"
- board text added: "BOOT"
- board text added: "GND"
- board text added: "MCzop 2025"
- board text added: "Mobile GS TRX board rev. 0"
- board text added: "RESET"
- board text added: "SBAND UHF"
- board text added: "SWC"
- board text added: "SWD"
- board text added: "SWDIO"

Commit message: Update designators
Other:
- board text added: "VEXT"
Changed lines of the file:
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@@
 			(psa4output no)
 			(plot_black_and_white yes)
-			(plotinvisibletext no)
 			(sketchpadsonfab no)
 			(plotpadnumbers no)
@@
 		(tags "Integrated Circuit")
 		(property "Reference" "U5"
-			(at 0 0 90)
+			(at 1.2 3.5 0)
 			(layer "F.SilkS")
 			(effects
@@
 		(tags "Integrated Circuit")
 		(property "Reference" "U4"
-			(at 0 0 0)
+			(at 3.65 -2.7 0)
 			(layer "F.SilkS")
 			(effects
@@
 			)
 			(justify left bottom)
+		)
+	)
+	(gr_text "VEXT\n"
+		(at 136 105 270)
+		(layer "F.SilkS" knockout)
+		(effects
+			(font
+				(size 1 1)
+				(thickness 0.2)
+				(bold yes)
+			)
+			(justify left bottom)
